File: hw/opensda.sch (KiCad schematic (older format))
At the start: 26 parts, among them J1 UX60SC-MB-5S8, P1 CONN_02X05, P2 CONN_01X02, U1 K20P32M50SF0, U2 74LVC125, Y1 Crystal_GND24

Commit message: Schematic complete except for decoupling
Parts:
- removed P2: CONN_01X02, symbol CONN_01X02
- removed TP1: TEST, symbol TEST
- added R209, R212: 0, symbol R_Small
- added TP201: TEST_1P, symbol TEST_1P
- Y201: renamed from Y1; value Crystal_GND24 -> 8MHz
- gave numbers to parts that had none: 2
- renumbered C1 to C201, C2 to C202, C4 to C203, C3 to C204, C5 to C205, D1 to D201, D2 to D202, J1 to J201, L1 to L201, L2 to L202, P1 to P201, R1 to R201, R2 to R202, R3 to R203, R4 to R206, R5 to R207, R6 to R208, R7 to R210, R8 to R211, U1 to U201, U2 to U202
Connections:
- wire segments 152 -> 130
Other:
- moved on the sheet: C201, C205, L202

Commit message: Define some footprints
Parts:
- C201, C202, C203, C204, C205, L201, L202, R201, R202, R203, R204, R205, R206, R207, R208, R210, R211: footprint (none) -> Resistors_SMD:R_0603_HandSoldering
- D201: footprint (none) -> LEDs:LED_0603
- D202: footprint (none) -> TO_SOT_Packages_SMD:SOT-23_Handsoldering
- P201: footprint (none) -> Pin_Headers:Pin_Header_Straight_2x05_Pitch1.27mm_SMD
- R209, R212: footprint (none) -> Resistors_SMD:R_0402
- TP201: footprint (none) -> Measurement_Points:Measurement_Point_Round-TH_Small
- U201: footprint 32 QFN -> Housings_DFN_QFN:QFN-32-1EP_5x5mm_Pitch0.5mm
Changed lines of the file:
@@
 F 0 "U201" H 4650 800 50  0000 C CNN
 F 1 "K20P32M50SF0" H 4650 700 50  0000 C CNN
-F 2 "32 QFN" H 4650 600 50  0001 C CNN
+F 2 "Housings_DFN_QFN:QFN-32-1EP_5x5mm_Pitch0.5mm" H 4650 600 50  0001 C CNN
 F 3 "K20P32M50SF0-782540.pdf" H 6250 4000 50  0001 C CNN
 	1    6200 2650
@@
 F 0 "L201" V 1350 3450 50  0000 C CNN
 F 1 "330 Ohm" V 1475 3450 50  0000 C CNN
-F 2 "" H 1400 3450 50  0001 C CNN
+F 2 "Resistors_SMD:R_0603_HandSoldering" H 1400 3450 50  0001 C CNN
 F 3 "" H 1400 3450 50  0000 C CNN
 	1    1400 3450
@@
 F 0 "L202" V 2100 1800 50  0000 C CNN
 F 1 "330 Ohm" V 2225 1800 50  0000 C CNN
-F 2 "" H 2150 1800 50  0001 C CNN
+F 2 "Resistors_SMD:R_0603_HandSoldering" H 2150 1800 50  0001 C CNN
 F 3 "" H 2150 1800 50  0000 C CNN
 	1    2150 1800
@@
 F 0 "C201" H 2860 2120 50  0000 L CNN
 F 1 "1.0 uF" H 2860 1970 50  0000 L CNN
-F 2 "" H 2850 2050 50  0001 C CNN
+F 2 "Resistors_SMD:R_0603_HandSoldering" H 2850 2050 50  0001 C CNN
 F 3 "" H 2850 2050 50  0000 C CNN
 	1    2850 2050
@@
 F 0 "R206" V 2600 2350 50  0000 L CNN
 F 1 "33" V 2600 2650 50  0000 L CNN
-F 2 "" H 2650 2550 50  0001 C CNN
+F 2 "Resistors_SMD:R_0603_HandSoldering" H 2650 2550 50  0001 C CNN
 F 3 "" H 2650 2550 50  0000 C CNN
 	1    2650 2550
@@
 F 0 "R207" V 2600 2450 50  0000 L CNN
 F 1 "33" V 2600 2750 50  0000 L CNN
-F 2 "" H 2650 2650 50  0001 C CNN
+F 2 "Resistors_SMD:R_0603_HandSoldering" H 2650 2650 50  0001 C CNN
 F 3 "" H 2650 2650 50  0000 C CNN
 	1    2650 2650
@@
 F 0 "D202" H 2400 3100 50  0000 C CNN
 F 1 "GSOT05C-GS08" H 2350 3300 50  0000 C CNN
-F 2 "" H 2350 3200 50  0001 C CNN
+F 2 "TO_SOT_Packages_SMD:SOT-23_Handsoldering" H 2350 3200 50  0001 C CNN
 F 3 "" H 2350 3200 50  0000 C CNN
 	1    2350 3200
@@
 F 0 "R202" H 1750 6500 50  0000 L CNN
 F 1 "4.7k" H 1750 6400 50  0000 L CNN
-F 2 "" H 1700 6450 50  0001 C CNN
+F 2 "Resistors_SMD:R_0603_HandSoldering" H 1700 6450 50  0001 C CNN
 F 3 "" H 1700 6450 50  0000 C CNN
 	1    1700 6450
@@
 F 0 "R203" H 1730 6770 50  0000 L CNN
 F 1 "10k" H 1730 6710 50  0000 L CNN
-F 2 "" H 1700 6750 50  0001 C CNN
+F 2 "Resistors_SMD:R_0603_HandSoldering" H 1700 6750 50  0001 C CNN
 F 3 "" H 1700 6750 50  0000 C CNN
 	1    1700 6750
@@
 F 0 "P201" H 3000 6950 50  0000 C CNN
 F 1 "CONN_02X05" H 3000 6350 50  0000 C CNN
-F 2 "" H 3000 5450 50  0001 C CNN
+F 2 "Pin_Headers:Pin_Header_Straight_2x05_Pitch1.27mm_SMD" H 3000 5450 50  0001 C CNN
 F 3 "" H 3000 5450 50  0000 C CNN
 	1    3000 6650
@@
 F 0 "R208" H 3380 6220 50  0000 L CNN
 F 1 "10k" H 3380 6160 50  0000 L CNN
-F 2 "" H 3350 6200 50  0001 C CNN
+F 2 "Resistors_SMD:R_0603_HandSoldering" H 3350 6200 50  0001 C CNN
 F 3 "" H 3350 6200 50  0000 C CNN
 	1    3350 6200
@@
 F 0 "R210" V 9050 1250 50  0000 L CNN
 F 1 "10k" V 9050 1500 50  0000 L CNN
-F 2 "" H 9000 1400 50  0001 C CNN
+F 2 "Resistors_SMD:R_0603_HandSoldering" H 9000 1400 50  0001 C CNN
 F 3 "" H 9000 1400 50  0000 C CNN
 	1    9000 1400
@@
 F 0 "R211" V 9050 2250 50  0000 L CNN
 F 1 "10k" V 9050 2500 50  0000 L CNN
-F 2 "" H 9000 2400 50  0001 C CNN
+F 2 "Resistors_SMD:R_0603_HandSoldering" H 9000 2400 50  0001 C CNN
 F 3 "" H 9000 2400 50  0000 C CNN
 	1    9000 2400
@@
 F 0 "C203" H 5210 6770 50  0000 L CNN
 F 1 "22 pF" H 5210 6620 50  0000 L CNN
-F 2 "" H 5200 6700 50  0001 C CNN
+F 2 "Resistors_SMD:R_0603_HandSoldering" H 5200 6700 50  0001 C CNN
 F 3 "" H 5200 6700 50  0000 C CNN
 	1    5200 6700
@@
 F 0 "C202" H 4310 6770 50  0000 L CNN
 F 1 "22 pF" H 4310 6620 50  0000 L CNN
-F 2 "" H 4300 6700 50  0001 C CNN
+F 2 "Resistors_SMD:R_0603_HandSoldering" H 4300 6700 50  0001 C CNN
 F 3 "" H 4300 6700 50  0000 C CNN
 	1    4300 6700
@@
 F 0 "D201" V 1000 6700 50  0000 C CNN
 F 1 "LED_GREEN" V 900 6550 50  0000 C CNN
-F 2 "" H 900 6800 50  0001 C CNN
+F 2 "LEDs:LED_0603" H 900 6800 50  0001 C CNN
 F 3 "" H 900 6800 50  0000 C CNN
 	1    900  6800
@@
 F 0 "R201" H 750 6400 50  0000 L CNN
 F 1 "220" H 700 6500 50  0000 L CNN
-F 2 "" H 900 6450 50  0001 C CNN
+F 2 "Resistors_SMD:R_0603_HandSoldering" H 900 6450 50  0001 C CNN
 F 3 "" H 900 6450 50  0000 C CNN
 	1    900  6450
@@
 F 0 "C204" V 5400 700 50  0000 L CNN
 F 1 "1.0 uF" V 5400 900 50  0000 L CNN
-F 2 "" H 5450 850 50  0001 C CNN
+F 2 "Resistors_SMD:R_0603_HandSoldering" H 5450 850 50  0001 C CNN
 F 3 "" H 5450 850 50  0000 C CNN
 	1    5450 850
@@
 F 0 "C205" H 8510 4420 50  0000 L CNN
 F 1 "2.2 uF" H 8510 4270 50  0000 L CNN
-F 2 "" H 8500 4350 50  0001 C CNN
+F 2 "Resistors_SMD:R_0603_HandSoldering" H 8500 4350 50  0001 C CNN
 F 3 "" H 8500 4350 50  0000 C CNN
 	1    8500 4350
@@
 F 0 "R204" H 2150 6500 50  0000 L CNN
 F 1 "4.7k" H 2150 6400 50  0000 L CNN
-F 2 "" H 2100 6450 50  0001 C CNN
+F 2 "Resistors_SMD:R_0603_HandSoldering" H 2100 6450 50  0001 C CNN
 F 3 "" H 2100 6450 50  0000 C CNN
 	1    2100 6450
@@
 F 0 "R205" H 2150 6800 50  0000 L CNN
 F 1 "10k" H 2150 6700 50  0000 L CNN
-F 2 "" H 2100 6750 50  0001 C CNN
+F 2 "Resistors_SMD:R_0603_HandSoldering" H 2100 6750 50  0001 C CNN
 F 3 "" H 2100 6750 50  0000 C CNN
 	1    2100 6750
@@
 F 0 "R212" V 10300 800 50  0000 L CNN
 F 1 "0" V 10300 1050 50  0000 L CNN
-F 2 "" H 10250 950 50  0001 C CNN
+F 2 "Resistors_SMD:R_0402" H 10250 950 50  0001 C CNN
 F 3 "" H 10250 950 50  0000 C CNN
 	1    10250 950
@@
 F 0 "R209" V 8850 4000 50  0000 L CNN
 F 1 "0" V 8850 4250 50  0000 L CNN
-F 2 "" H 8800 4150 50  0001 C CNN
+F 2 "Resistors_SMD:R_0402" H 8800 4150 50  0001 C CNN
 F 3 "" H 8800 4150 50  0000 C CNN
 	1    8800 4150
@@
 F 0 "TP201" H 2100 2650 50  0000 C CNN
 F 1 "TEST_1P" H 2100 2650 50  0001 C CNN
-F 2 "" H 2300 2450 50  0001 C CNN
+F 2 "Measurement_Points:Measurement_Point_Round-TH_Small" H 2300 2450 50  0001 C CNN
 F 3 "" H 2300 2450 50  0000 C CNN
 	1    2100 2450
