File: hw/usb.sch (KiCad schematic (older format))
At the start: 16 parts, among them U201 74LVC1G32, U202 USB_TYPE_C, U203 PI3USB3102-334678, U204 USB_TYPE_C

Commit message: Add some more footprints
Parts:
- U201: footprint (none) -> TO_SOT_Packages_SMD:SOT-353_SC-70-5_Handsoldering
- U203: footprint TQFN-32 -> horu:TQFN32_ZL32
Changed lines of the file:
@@
 F 0 "U201" H 2500 1750 50  0000 C CNN
 F 1 "74LVC1G32" H 2500 1650 50  0000 C CNN
-F 2 "" H 2500 1700 50  0001 C CNN
+F 2 "TO_SOT_Packages_SMD:SOT-353_SC-70-5_Handsoldering" H 2500 1700 50  0001 C CNN
 F 3 "" H 2500 1700 50  0000 C CNN
 	1    2500 1700
@@
 F 0 "U203" H 5550 4600 50  0000 C CNN
 F 1 "PI3USB3102-334678" H 5550 4800 50  0000 C CNN
-F 2 "TQFN-32" H 5550 4700 50  0001 C CNN
+F 2 "horu:TQFN32_ZL32" H 5550 4700 50  0001 C CNN
 F 3 "DOCUMENTATION" H 5550 4700 50  0001 C CNN
 	1    5550 4600
