File: hw/horu.sch (KiCad schematic (older format))
At the start: 33 parts, among them P1 CONN_01X06, P2 DNP, P3 CONN_01X30_2SHIELD, P4 CONN_01X06, P5 CONN_02X05, U1 KL25P80M48SF0, Y1 8MHz

Commit message: Update to KiCad 5.1.5 & replace EOL capacitors
Parts:
- C1, C4, C5: symbol C_Small -> horu-rescue:C_Small; DstPart 81-GRM39R105K16 -> 603-CC603KPX7R7BB105; manf# GRM188R61C105KA93D -> CC0603KPX7R7BB105
- C2, C3: symbol C_Small -> horu-rescue:C_Small
- C6: symbol C_Small -> horu-rescue:C_Small; DstPart 81-GRM188R61C225KE15 -> 810-C168X7S1C225K8AC; manf# GRM188R61C225KE15D -> C1608X7S1C225K080AC
- D1, D2, D3, D4: symbol LED -> horu-rescue:LED
- D5: symbol D_Zener_x2_ACom_KKA -> horu:D_Zener_x2_ACom_KKA
- JP1: symbol Jumper_NC_Dual -> horu-rescue:Jumper_NC_Dual
- L1, L2: symbol L -> horu-rescue:L
- P1, P4: symbol CONN_01X06 -> horu-rescue:CONN_01X06
- P2: symbol USB_OTG -> horu-rescue:USB_OTG
- P3: symbol CONN_01X30_2SHIELD -> horu:CONN_01X30_2SHIELD
- P5: symbol CONN_02X05 -> horu-rescue:CONN_02X05
- R1, R2, R3, R4, R5, R6, R7, R8: symbol R_Small -> horu-rescue:R_Small
- TP1, TP2, TP3, TP4: symbol TEST_1P -> horu-rescue:TEST_1P
- U1: value KL25P80M48SF0 -> MKL25Z128VLK4; symbol KL25P80M48SF0 -> KL25P80M48SF0:KL25P80M48SF0
- Y1: symbol Crystal_GND24 -> horu-rescue:Crystal_GND24
Connections:
- wire segments 180 -> 205
